File: board/MiniMain-esp32-s2/MiniMain-esp32-s2.kicad_sch (KiCad schematic)
At the start: 41 parts, among them IC1 ESP32-S2-MINI-1-N4R2, J1 USB4105-GF-A, J10 Conn_01x03_Male, J2 Conn_01x04, J3 Conn_01x16, J5 Conn_01x12, J8 Conn_01x02, Q1 DMP3130LQ-7, SW1 SW_Push, SW2 SW_Push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

Commit message: Rev 2: Change Stemma QT compatible port from transistor controlled power to just +3.3V. Remove copper pour under the ESP32-S2 antenna. Perhaps look at changing the isolated input pull-up from 150 ohms to 1k ohms.
Parts:
- removed C5: 1uF, Capacitor_SMD:C_0603_1608Metric, symbol Device:C
- removed Q1: DMP3130LQ-7, Package_TO_SOT_SMD:SOT-23, symbol Transistor_FET:AO3401A
- removed R9: 100k, Resistor_SMD:R_0603_1608Metric, symbol Device:R
Connections:
- net VDEVICE is gone; now on net +3V3: J2.2 (Pin_2)
- net I2C_PWR: no longer names the net of IC1.11 (IO7)
- no-connect marks 10 -> 11
Other:
- note added: "Look at 1k"
